File: kicad/dhd/dhd.kicad_pcb (KiCad board)
At the start: 2 copper layers, 66 x 69.1 mm, 9 parts, among them J1 Motor, J2 Pot

Commit message: Submitted KiCad design v1
Connections:
- net Net-(A1-AGND) renamed /3
- A1 pad 19: /IN2 -> /IN1
- A1 pad 20: /IN1 -> /IN2
- A1 pad 26: Net-(A1-GPIO20) -> unconnected-(A1-GPIO20-Pad26)
- A1 pad 31: unconnected-(A1-GPIO26_ADC0-Pad31) -> /2
- J2 pad 2: unconnected-(J2-Pin_2-Pad2) -> /T
- J2 pad 3: Net-(A1-GPIO20) -> /2
Routing:
- net Net-(A1-GPIO20): track 47.8 -> 0.00 mm
- net /2: track 0.00 -> 42.5 mm
- net /IN1: track 44.8 -> 55.8 mm
- net /IN2: track 45.9 -> 48.1 mm
Changed lines of the file:
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@@
 	)
 	(setup
+		(stackup
+			(layer "F.SilkS"
+				(type "Top Silk Screen")
+			)
+			(layer "F.Paste"
+				(type "Top Solder Paste")
+			)
+			(layer "F.Mask"
+				(type "Top Solder Mask")
+				(thickness 0.01)
+			)
+			(layer "F.Cu"
+				(type "copper")
+				(thickness 0.035)
+			)
+			(layer "dielectric 1"
+				(type "core")
+				(thickness 1.51)
+				(material "FR4")
+				(epsilon_r 4.5)
+				(loss_tangent 0.02)
+			)
+			(layer "B.Cu"
+				(type "copper")
+				(thickness 0.035)
+			)
+			(layer "B.Mask"
+				(type "Bottom Solder Mask")
+				(thickness 0.01)
+			)
+			(layer "B.Paste"
+				(type "Bottom Solder Paste")
+			)
+			(layer "B.SilkS"
+				(type "Bottom Silk Screen")
+			)
+			(copper_finish "None")
+			(dielectric_constraints no)
+		)
 		(pad_to_mask_clearance 0)
 		(allow_soldermask_bridges_in_footprints no)
@@
 			(layers "*.Cu" "*.Mask")
 			(remove_unused_layers no)
-			(net "/IN2")
+			(net "/IN1")
 			(pinfunction "GPIO14_19")
 			(pintype "bidirectional")
@@
 			(layers "*.Cu" "*.Mask")
 			(remove_unused_layers no)
-			(net "/IN1")
+			(net "/IN2")
 			(pinfunction "GPIO15_20")
 			(pintype "bidirectional")
@@
 			(layers "*.Cu" "*.Mask")
 			(remove_unused_layers no)
-			(net "Net-(A1-GPIO20)")
+			(net "unconnected-(A1-GPIO20-Pad26)")
 			(pinfunction "GPIO20_26")
 			(pintype "bidirectional")
@@
 			(layers "*.Cu" "*.Mask")
 			(remove_unused_layers no)
-			(net "unconnected-(A1-GPIO26_ADC0-Pad31)")
+			(net "/2")
 			(pinfunction "GPIO26_ADC0_31")
 			(pintype "bidirectional")
@@
 			(layers "*.Cu" "*.Mask")
 			(remove_unused_layers no)
-			(net "Net-(A1-AGND)")
+			(net "/3")
 			(pinfunction "AGND_33")
 			(pintype "power_out")
@@
 			(remove_unused_layers no)
 			(roundrect_rratio 0.147059)
-			(net "Net-(A1-AGND)")
+			(net "/3")
 			(pinfunction "Pin_1_1")
 			(pintype "passive")
@@
 			(layers "*.Cu" "*.Mask")
 			(remove_unused_layers no)
-			(net "unconnected-(J2-Pin_2-Pad2)")
+			(net "/T")
 			(pinfunction "Pin_2_2")
 			(pintype "passive")
@@
 			(layers "*.Cu" "*.Mask")
 			(remove_unused_layers no)
-			(net "Net-(A1-GPIO20)")
+			(net "/2")
 			(pinfunction "Pin_3_3")
 			(pintype "passive")
@@
 	)
 	(segment
-		(start 130.81 123.19)
-		(end 137.16 129.54)
+		(start 129.54 127)
+		(end 130.81 125.73)
 		(width 0.25)
 		(layer "F.Cu")
@@
 	)
 	(segment
-		(start 165.1 129.54)
-		(end 171.45 123.19)
+		(start 129.54 127)
+		(end 129.54 128.27)
+		(width 0.25)
+		(layer "F.Cu")
+		(net "/IN2")
+	)
+	(segment
+		(start 129.54 128.27)
+		(end 130.81 129.54)
 		(width 0.25)
 		(layer "F.Cu")
@@
 	)
 	(segment
-		(start 137.16 129.54)
+		(start 171.45 123.19)
 		(end 165.1 129.54)
 		(width 0.25)
@@
 	)
 	(segment
-		(start 166.37 130.81)
-		(end 135.89 130.81)
+		(start 165.1 129.54)
+		(end 130.81 129.54)
+		(width 0.25)
+		(layer "F.Cu")
+		(net "/IN2")
+	)
+	(segment
+		(start 127 124.46)
+		(end 128.27 123.19)
 		(width 0.25)
 		(layer "F.Cu")
@@
 	)
 	(segment
-		(start 135.89 130.81)
-		(end 130.81 125.73)
+		(start 127 128.27)
+		(end 127 124.46)
 		(width 0.25)
 		(layer "F.Cu")
@@
 	(segment
 		(start 166.37 130.81)
-		(end 171.45 125.73)
+		(end 129.54 130.81)
+		(width 0.25)
+		(layer "F.Cu")
+		(net "/IN1")
+	)
+	(segment
+		(start 129.54 130.81)
+		(end 127 128.27)
+		(width 0.25)
+		(layer "F.Cu")
+		(net "/IN1")
+	)
+	(segment
+		(start 128.27 123.19)
+		(end 130.81 123.19)
+		(width 0.25)
+		(layer "F.Cu")
+		(net "/IN1")
+	)
+	(segment
+		(start 171.45 125.73)
+		(end 166.37 130.81)
 		(width 0.25)
 		(layer "F.Cu")
@@
 	)
 	(segment
-		(start 165.1 90.17)
+		(start 161.29 100.33)
 		(end 165.1 96.52)
 		(width 0.5)
 		(layer "F.Cu")
-		(net "Net-(A1-GPIO20)")
+		(net "/2")
 	)
 	(segment
-		(start 172.72 87.63)
-		(end 171.45 88.9)
+		(start 171.47 81.3)
+		(end 172.72 82.55)
 		(width 0.5)
 		(layer "F.Cu")
-		(net "Net-(A1-GPIO20)")
+		(net "/2")
 	)
 	(segment
-		(start 168.91 81.3)
-		(end 171.47 81.3)
+		(start 172.72 87.63)
+		(end 171.45 88.9)
 		(width 0.5)
 		(layer "F.Cu")
-		(net "Net-(A1-GPIO20)")
+		(net "/2")
 	)
 	(segment
-		(start 165.1 96.52)
-		(end 148.59 113.03)
+		(start 148.59 100.33)
+		(end 161.29 100.33)
 		(width 0.5)
 		(layer "F.Cu")
-		(net "Net-(A1-GPIO20)")
+		(net "/2")
 	)
 	(segment
@@
 		(width 0.5)
 		(layer "F.Cu")
-		(net "Net-(A1-GPIO20)")
+		(net "/2")
 	)
 	(segment
-		(start 166.37 88.9)
-		(end 165.1 90.17)
+		(start 165.1 90.17)
+		(end 165.1 96.52)
 		(width 0.5)
 		(layer "F.Cu")
-		(net "Net-(A1-GPIO20)")
+		(net "/2")
 	)
 	(segment
-		(start 171.45 88.9)
-		(end 166.37 88.9)
+		(start 168.91 81.3)
+		(end 171.47 81.3)
 		(width 0.5)
 		(layer "F.Cu")
-		(net "Net-(A1-GPIO20)")
+		(net "/2")
 	)
 	(segment
-		(start 171.47 81.3)
-		(end 172.72 82.55)
+		(start 166.37 88.9)
+		(end 165.1 90.17)
+		(width 0.5)
+		(layer "F.Cu")
+		(net "/2")
+	)
+	(segment
+		(start 171.45 88.9)
+		(end 166.37 88.9)
 		(width 0.5)
 		(layer "F.Cu")
-		(net "Net-(A1-GPIO20)")
+		(net "/2")
 	)
 	(segment
@@
 		(width 1)
 		(layer "F.Cu")
-		(net "Net-(A1-AGND)")
+		(net "/3")
 	)
 	(segment
@@
 		(width 1)
 		(layer "F.Cu")
-		(net "Net-(A1-AGND)")
+		(net "/3")
 	)
 	(group ""
